Commit message: gazebo definition added to urdf ur5

File: urdf/ur5_egomo_table.urdf (robot description, URDF)
Before this commit: robot ur5, 25 links, 24 joints
Joints:
- joint robotiq_85_finger_left_1_joint: mimic joint=robotiq_85_finger_right_1_joint multiplier=-1 -> joint=robotiq_85_finger_right_1_joint multiplier=-1 offset=0; type revolute -> continuous
- joint robotiq_85_finger_left_3_joint: mimic joint=robotiq_85_finger_right_1_joint multiplier=-1 -> joint=robotiq_85_finger_right_1_joint multiplier=-1 offset=0; type revolute -> continuous
- joint robotiq_85_finger_left_4_joint: mimic joint=robotiq_85_finger_right_1_joint multiplier=1 -> joint=robotiq_85_finger_right_1_joint multiplier=1 offset=0; type revolute -> continuous
- joint robotiq_85_finger_right_1_joint: type revolute -> continuous
- joint robotiq_85_finger_right_3_joint: mimic joint=robotiq_85_finger_right_1_joint multiplier=1 -> joint=robotiq_85_finger_right_1_joint multiplier=1 offset=0; type revolute -> continuous
- joint robotiq_85_finger_right_4_joint: mimic joint=robotiq_85_finger_right_1_joint multiplier=-1 -> joint=robotiq_85_finger_right_1_joint multiplier=-1 offset=0; type revolute -> continuous
- joint shoulder_pan_joint: origin xyz=0.0 0.0 0.089159 rpy=0.0 0.0 0.0 -> xyz=0.0 0.0 0.089159 rpy=0.0 0.0 0.7853981625

Commit message: first test with new controller

File: urdf/ur5_egomo_table.urdf (robot description, URDF)
Before this commit: robot ur5, 25 links, 24 joints
Joints:
- joint shoulder_pan_joint: origin xyz=0.0 0.0 0.089159 rpy=0.0 0.0 0.7853981625 -> xyz=0.0 0.0 0.089159 rpy=0.0 0.0 0.0
