Commit message: new folder strukture

File: egomo_ur5/urdf/ur5_egomo_table.urdf (robot description, URDF)
Before this commit: robot ur5, 25 links, 24 joints
Links:
- link base_link: geometry collision mesh filename=package://egomo_ur5/meshes/ur5/collision/base.stl; visual mesh filename=package://egomo_ur5/meshes/ur5/visual/base.dae
- link camera_robotside: geometry collision mesh filename=package://egomo_ur5/meshes/egomo-1/collision/egomo-1.stl; visual mesh filename=package://egomo_ur5/meshes/egomo-1/visual/egomo-1.dae
- link forearm_link: geometry collision mesh filename=package://egomo_ur5/meshes/ur5/collision/forearm.stl; visual mesh filename=package://egomo_ur5/meshes/ur5/visual/forearm.dae
- link fts_robotside: geometry collision mesh filename=package://egomo_ur5/meshes/robotiq-ft300/collision/ft300.stl; visual mesh filename=package://egomo_ur5/meshes/robotiq-ft300/visual/ft300.dae
- link robotiq_85_base: geometry collision mesh filename=package://egomo_ur5/meshes/robotiq-2-finger-85/collision/gr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; visual mesh filename=package://egomo_ur5/meshes/robotiq-2-finger-85/visual/gripp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
- link robotiq_85_coupling: geometry collision mesh filename=package://egomo_ur5/meshes/robotiq-2-finger-85/collision/gr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; visual mesh filename=package://egomo_ur5/meshes/robotiq-2-finger-85/visual/gripp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
- link robotiq_85_finger_left_1: geometry collision mesh filename=package://egomo_ur5/meshes/robotiq-2-finger-85/collision/gr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; visual mesh filename=package://egomo_ur5/meshes/robotiq-2-finger-85/visual/gripp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
- link robotiq_85_finger_left_2: geometry collision mesh filename=package://egomo_ur5/meshes/robotiq-2-finger-85/collision/gr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; visual mesh filename=package://egomo_ur5/meshes/robotiq-2-finger-85/visual/gripp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
- link robotiq_85_finger_left_3: geometry collision mesh filename=package://egomo_ur5/meshes/robotiq-2-finger-85/collision/gr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; visual mesh filename=package://egomo_ur5/meshes/robotiq-2-finger-85/visual/gripp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
- link robotiq_85_finger_left_4: geometry collision mesh filename=package://egomo_ur5/meshes/robotiq-2-finger-85/collision/gr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; visual mesh filename=package://egomo_ur5/meshes/robotiq-2-finger-85/visual/gripp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
- link robotiq_85_finger_right_1: geometry collision mesh filename=package://egomo_ur5/meshes/robotiq-2-finger-85/collision/gr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; visual mesh filename=package://egomo_ur5/meshes/robotiq-2-finger-85/visual/gripp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
- link robotiq_85_finger_right_2: geometry collision mesh filename=package://egomo_ur5/meshes/robotiq-2-finger-85/collision/gr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; visual mesh filename=package://egomo_ur5/meshes/robotiq-2-finger-85/visual/gripp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
- link robotiq_85_finger_right_3: geometry collision mesh filename=package://egomo_ur5/meshes/robotiq-2-finger-85/collision/gr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; visual mesh filename=package://egomo_ur5/meshes/robotiq-2-finger-85/visual/gripp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
- link robotiq_85_finger_right_4: geometry collision mesh filename=package://egomo_ur5/meshes/robotiq-2-finger-85/collision/gr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; visual mesh filename=package://egomo_ur5/meshes/robotiq-2-finger-85/visual/gripp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
- link shoulder_link: geometry collision mesh filename=package://egomo_ur5/meshes/ur5/collision/shoulder.stl; visual mesh filename=package://egomo_ur5/meshes/ur5/visual/shoulder.dae
- link upper_arm_link: geometry collision mesh filename=package://egomo_ur5/meshes/ur5/collision/upper_arm.stl; visual mesh filename=package://egomo_ur5/meshes/ur5/visual/upper_arm.dae
- link wrist_1_link: geometry collision mesh filename=package://egomo_ur5/meshes/ur5/collision/wrist_1.stl; visual mesh filename=package://egomo_ur5/meshes/ur5/visual/wrist_1.dae
- link wrist_2_link: geometry collision mesh filename=package://egomo_ur5/meshes/ur5/collision/wrist_2.stl; visual mesh filename=package://egomo_ur5/meshes/ur5/visual/wrist_2.dae
- link wrist_3_link: geometry collision mesh filename=package://egomo_ur5/meshes/ur5/collision/wrist_3.stl; visual mesh filename=package://egomo_ur5/meshes/ur5/visual/wrist_3.dae
Joints:
- joint ee_fixed_joint: origin xyz=0.0 0.0823 0.0 rpy=-1.570796326795 0.0 0 -> xyz=0.0 ${wrist_3_length} 0.0 rpy=-1.570796326795 0.0 0
- joint elbow_joint: origin xyz=0.0 -0.1197 0.425 rpy=0.0 0.0 0.0 -> xyz=0.0 ${elbow_offset} ${upper_arm_length} rpy=0.0 0.0 0.0
- joint shoulder_pan_joint: origin xyz=0.0 0.0 0.089159 rpy=0.0 0.0 0.0 -> xyz=0.0 0.0 ${shoulder_height} rpy=0.0 0.0 0.0
- joint wrist_1_joint: origin xyz=0.0 0.0 0.39225 rpy=0.0 1.570796326795 0.0 -> xyz=0.0 0.0 ${forearm_length} rpy=0.0 ${pi / 2.0} 0.0
- joint wrist_2_joint: origin xyz=0.0 0.093 0.0 rpy=0.0 0.0 0.0 -> xyz=0.0 ${wrist_1_length} 0.0 rpy=0.0 0.0 0.0
- joint wrist_3_joint: origin xyz=0.0 0.0 0.09465 rpy=0.0 0.0 0.0 -> xyz=0.0 0.0 ${wrist_2_length} rpy=0.0 0.0 0.0

Commit message: added urdf example

File: egomo_ur5/urdf/ur5_egomo_table.urdf (robot description, URDF)
Before this commit: robot ur5, 25 links, 24 joints
Links:
- removed link base
Joints:
- removed joint base_link-base_fixed_joint
- joint ee_fixed_joint: origin xyz=0.0 ${wrist_3_length} 0.0 rpy=-1.570796326795 0.0 0 -> xyz=0.0 0.0823 0.0 rpy=-1.570796326795 0.0 0
- joint elbow_joint: origin xyz=0.0 ${elbow_offset} ${upper_arm_length} rpy=0.0 0.0 0.0 -> xyz=0.0 -0.1197 0.425 rpy=0.0 0.0 0.0
- joint shoulder_pan_joint: origin xyz=0.0 0.0 ${shoulder_height} rpy=0.0 0.0 0.0 -> xyz=0.0 0.0 0.089159 rpy=0.0 0.0 0.0
- joint wrist_1_joint: origin xyz=0.0 0.0 ${forearm_length} rpy=0.0 ${pi / 2.0} 0.0 -> xyz=0.0 0.0 0.39225 rpy=0.0 1.57079632679 0.0
- joint wrist_2_joint: limit lower=-${pi} upper=${pi} effort=28.0 velocity=3.15 -> lower=-3.14159265359 upper=3.14159265359 effort=28.0 velocity=3.15; origin xyz=0.0 ${wrist_1_length} 0.0 rpy=0.0 0.0 0.0 -> xyz=0.0 0.093 0.0 rpy=0.0 0.0 0.0
- joint wrist_3_joint: limit lower=-${pi} upper=${pi} effort=28.0 velocity=3.15 -> lower=-3.14159265359 upper=3.14159265359 effort=28.0 velocity=3.15; origin xyz=0.0 0.0 ${wrist_2_length} rpy=0.0 0.0 0.0 -> xyz=0.0 0.0 0.09465 rpy=0.0 0.0 0.0

File: egomo_ur5/urdf/ur5_egomo_table_ori.urdf.xacro (robot description, xacro)
@@ -27,5 +27,5 @@
 -->
   </gazebo>
-<property name="pi" value="3.1415926535898" />3.14159265359
+<property name="pi" value="3.1415926535898" />
   <!-- Inertia parameters -->
   <property name="base_mass" value="4.0" />  <!-- This mass might be incorrect -->
@@ -49,66 +49,16 @@
     d = [0.089159,  0.00000,  0.00000,  0.10915,  0.09465,  0.0823]
     alpha = [ 1.570796327, 0, 0, 1.570796327, -1.570796327, 0 ]
-    theta = [0, -1.570796327, 0, -1.570796327, 0, 0]
+    q_home_offset = [0, -1.570796327, 0, -1.570796327, 0, 0]
     joint_direction = [-1, -1, 1, 1, 1, 1]
     mass = [3.7000, 8.3930, 2.2750, 1.2190, 1.2190, 0.1879]
     center_of_mass = [ [0, -0.02561, 0.00193], [0.2125, 0, 0.11336], [0.11993, 0.0, 0.0265], [0, -0.0018, 0.01634], [0, 0.0018,0.01634], [0, 0, -0.001159] ]
   -->
-  <property name="theta_1" value="0.0" />
   <property name="ur5_d1" value="0.089159" />
-  <property name="ur5_a1" value="0.0" />
-  <property name="alpha_1" value="${pi/2}" />
-  <property name="theta_2" value="-${pi/2}" />
-  <property name="ur5_d2" value="0.0" />
   <property name="ur5_a2" value="-0.42500" />
-  <property name="alpha_2" value="0.0" />
-  <property name="theta_3" value="0.0" />
-  <property name="ur5_d3" value="0.0" />
   <property name="ur5_a3" value="-0.39225" />
-  <property name="alpha_3" value="0.0" />
-  <property name="theta_4" value="-${pi/2}" />
   <property name="ur5_d4" value="0.10915" />
-  <property name="ur5_a4" value="0.0" />
-  <property name="alpha_4" value="${pi/2}" />
-  <property name="theta_5" value="0.0" />
   <property name="ur5_d5" value="0.09465" />
-  <property name="ur5_a5" value="0.0" />
-  <property name="alpha_5" value="-${pi/2}" />
-  <property name="theta_6" value="0.0" />
   <property name="ur5_d6" value="0.0823" />
-  <property name="ur5_a6" value="0.0" />
-  <property name="alpha_6" value="0.0" />
-<!--
-Joint 0(theta, d, a, alpha)-0.00205442 0.089159 0 1.57718
-Joint 1(theta, d, a, alpha)-0.000123686 0 0.425 -0.00201947
-Joint 2(theta, d, a, alpha)-0.000189364 0 0.39225 -0.00944871
-Joint 3(theta, d, a, alpha)0.000488426 -0.10915 0 1.57342
-Joint 4(theta, d, a, alpha)-0.000123914 0.09465 0 -1.57255
-Joint 5(theta, d, a, alpha)3.14254 -0.0823 0 3.14331
-  <property name="theta_1" value="-0.00205442" />
-  <property name="ur5_d1" value="0.089159" />
-  <property name="ur5_a1" value="0.0" />
-  <property name="alpha_1" value="1.57718" />
-  <property name="theta_2" value="-0.000123686" />
-  <property name="ur5_d2" value="0.0" />
-  <property name="ur5_a2" value="0.42500" />
-  <property name="alpha_2" value="-0.00201947" />
-  <property name="theta_3" value="-0.000189364" />
-  <property name="ur5_d3" value="0.0" />
-  <property name="ur5_a3" value="0.39225" />
-  <property name="alpha_3" value="-0.00944871" />
-  <property name="theta_4" value="-0.000488426" />
-  <property name="ur5_d4" value="-0.10915" />
-  <property name="ur5_a4" value="0.0" />
-  <property name="alpha_4" value="1.57342" />
-  <property name="theta_5" value="-0.000123914" />
-  <property name="ur5_d5" value="0.09465" />
-  <property name="ur5_a5" value="0.0" />
-  <property name="alpha_5" value="-1.57255" />
-  <property name="theta_6" value="3.14254" />
-  <property name="ur5_d6" value="-0.0823" />
-  <property name="ur5_a6" value="0.0" />
-  <property name="alpha_6" value="3.14331" />
--->
- <!-- Arbitrary offsets for shoulder/elbow joints -->
+  <!-- Arbitrary offsets for shoulder/elbow joints -->
   <property name="shoulder_offset" value="0.13585" />  <!-- measured from model -->
   <property name="elbow_offset" value="-0.1197" /> <!-- measured from model -->
@@ -153,15 +103,14 @@
     </inertial>
   </link>
-  <joint name="shoulder_pan_joint" type="revolute"> <!--Joint 1-->
+  <joint name="shoulder_pan_joint" type="revolute">
     <parent link="base_link"/>
-    <child link="shoulder_linka"/>
-    <origin rpy="0.0 0.0 ${theta_1 }" xyz="0.0 0.0 ${ur5_d1}"/><!--origin rpy="0.0 0.0 0.7853981625" xyz="0.0 0.0 0.089159"/-->
+    <child link="shoulder_link"/>
+    <origin rpy="0.0 0.0 0.0" xyz="0.0 0.0 ${shoulder_height}"/><!--origin rpy="0.0 0.0 0.7853981625" xyz="0.0 0.0 0.089159"/-->
     <axis xyz="0 0 1"/>
     <limit effort="150.0" lower="-3.14159265" upper="3.14159265" velocity="3.15"/>
     <dynamics damping="0.0" friction="0.0"/>
   </joint>
-  <link name="shoulder_linka">
-    <visual>
-	<origin xyz="0 0 0" rpy="0.0 0 0" />
+  <link name="shoulder_link">
+    <visual>
       <geometry>
         <mesh filename="package://egomo_ur5/meshes/ur5/visual/shoulder.dae"/>
@@ -182,13 +131,16 @@
     </inertial>
   </link>
- <joint name="shoulder_pan_joint_F" type="fixed"> <!--Joint 1-->
-    <parent link="shoulder_linka"/>
-    <child link="shoulder_link"/>
-    <origin rpy="${alpha_1} 0.0 0.0" xyz="${ur5_a1} 0.0 0.0"/><!--origin rpy="0.0 0.0 0.7853981625" xyz="0.0 0.0 0.089159"/-->
-  </joint>
-  <link name="shoulder_link">
-    <visual>
-      <geometry>
-        <box size="0 0 0" />
+  <joint name="shoulder_lift_joint" type="revolute">
+    <parent link="shoulder_link"/>
+    <child link="upper_arm_link"/>
+    <origin rpy="0.0 1.570796326795 0.0" xyz="0.0 0.13585 0.0"/>
+    <axis xyz="0 1 0"/>
+    <limit effort="150.0" lower="-3.14159265" upper="-0.1" velocity="3.15"/>
+    <dynamics damping="0.0" friction="0.0"/>
+  </joint>
+  <link name="upper_arm_link">
+    <visual>
+      <geometry>
+        <mesh filename="package://egomo_ur5/meshes/ur5/visual/upper_arm.dae"/>
       </geometry>
       <material name="LightGrey">
@@ -196,33 +148,5 @@
       </material>
     </visual>
-     <inertial>
-        <origin xyz="0 0 0" rpy="0 0 0" />
-        <mass value="1" />
-        <inertia
-          ixx="1.0" ixy="0.0" ixz="0.0"
-          iyy="1.0" iyz="0.0"
-          izz="1.0" />
-    </inertial>
-  </link>
-  <joint name="shoulder_lift_joint" type="revolute"><!--Joint 2-->
-    <parent link="shoulder_link"/>
-    <child link="upper_arm_linka"/>
- <origin rpy="0.0 0.0 ${theta_2}" xyz="0.0 0.0 ${ur5_d2+elbow_offset}"/><!--Joint 2-->
-    <axis xyz="0 0 -1"/>
-    <limit effort="150.0" lower="-3.14159265" upper="-0.1" velocity="3.15"/>
-    <dynamics damping="0.0" friction="0.0"/>
-  </joint>
-  <link name="upper_arm_linka">
-    <visual>
-	<origin xyz="0 0 0" rpy="-${pi/2} 0 0" />
-      <geometry>
-        <mesh filename="package://egomo_ur5/meshes/ur5/visual/upper_arm.dae"/>
-      </geometry>
-      <material name="LightGrey">
-        <color rgba="0.7 0.7 0.7 1.0"/>
-      </material>
-    </visual>
-    <collision>
-<origin xyz="0 0 0" rpy="-${pi/2} 0 0" />
+    <collision>
       <geometry>
         <mesh filename="package://egomo_ur5/meshes/ur5/collision/upper_arm.stl"/>
@@ -235,13 +159,17 @@
     </inertial>
   </link>
-<joint name="upper_arm_link_F" type="fixed"> <!--Joint 1-->
-    <parent link="upper_arm_linka"/>
-    <child link="upper_arm_link"/>
-    <origin rpy="${alpha_2} 0.0 0.0" xyz="0.0 ${-ur5_a2} 0.0 "/><!--origin rpy="0.0 0.0 0.7853981625" xyz="0.0 0.0 0.089159"/-->
-  </joint>
-  <link name="upper_arm_link">
-    <visual>
-      <geometry>
-        <box size="0 0 0" />
+  <joint name="elbow_joint" type="revolute">
+    <parent link="upper_arm_link"/>
+    <child link="forearm_link"/>
+    <origin xyz="0.0 ${elbow_offset} ${upper_arm_length}" rpy="0.0 0.0 0.0" />
+<!--origin rpy="0.0 0.0 0.0" xyz="0.0 -0.1197 0.425"/-->
+    <axis xyz="0 1 0"/>
+    <limit effort="150.0" lower="-3" upper="3" velocity="3.15"/> <!-- +/- 175 deg -->
+    <dynamics damping="0.0" friction="0.0"/>
+  </joint>
+  <link name="forearm_link">
+    <visual>
+      <geometry>
+        <mesh filename="package://egomo_ur5/meshes/ur5/visual/forearm.dae"/>
       </geometry>
       <material name="LightGrey">
@@ -249,34 +177,5 @@
       </material>
     </visual>
-     <inertial>
-        <origin xyz="0 0 0" rpy="0 0 0" />
-        <mass value="1" />
-        <inertia
-          ixx="1.0" ixy="0.0" ixz="0.0"
-          iyy="1.0" iyz="0.0"
-          izz="1.0" />
-    </inertial>
-  </link>
-  <joint name="elbow_joint" type="revolute"> <!--Joint 3-->
-    <parent link="upper_arm_link"/>
-    <child link="forearm_linka"/>
- <origin rpy="0.0 0.0 ${theta_3}" xyz="0.0 0.0 ${ur5_d3-elbow_offset}"/>
-<!--origin rpy="0.0 0.0 0.0" xyz="0.0 -0.1197 0.425"/-->
-    <axis xyz="0 0 -1"/>
-    <limit effort="150.0" lower="-3" upper="3" velocity="3.15"/> <!-- +/- 175 deg -->
-    <dynamics damping="0.0" friction="0.0"/>
-  </joint>
-<link name="forearm_linka">
- <visual>
-	<origin xyz="0 0 0" rpy="-${pi/2} 0 0" />
-      <geometry>
-        <mesh filename="package://egomo_ur5/meshes/ur5/visual/forearm.dae"/>
-      </geometry>
-      <material name="LightGrey">
-        <color rgba="0.7 0.7 0.7 1.0"/>
-      </material>
-    </visual>
-    <collision>
-<origin xyz="0 0 0" rpy="-${pi/2} 0 0" />
+    <collision>
       <geometry>
         <mesh filename="package://egomo_ur5/meshes/ur5/collision/forearm.stl"/>
@@ -288,14 +187,18 @@
       <inertia ixx="0.049443313556" ixy="0.0" ixz="0.0" iyy="0.049443313556" iyz="0.0" izz="0.004095"/>
     </inertial>
- </link>
-<joint name="elbow_joint_F" type="fixed"> <!--Joint 1-->
-    <parent link="forearm_linka"/>
-    <child link="forearm_link"/>
-    <origin rpy="${alpha_3} 0.0 0.0" xyz="0.0 ${-ur5_a3} 0.0"/><!--origin rpy="0.0 0.0 0.7853981625" xyz="0.0 0.0 0.089159"/-->
-  </joint>
-  <link name="forearm_link">
-    <visual>
-      <geometry>
-        <box size="0 0 0" />
+  </link>
+  <joint name="wrist_1_joint" type="revolute">
+    <parent link="forearm_link"/>
+    <child link="wrist_1_link"/>
+    <origin xyz="0.0 0.0 ${forearm_length}" rpy="0.0 ${pi / 2.0} 0.0" />
+    <!--origin rpy="0.0 1.570796326795 0.0" xyz="0.0 0.0 0.39225"/-->
+    <axis xyz="0 1 0"/>
+    <limit effort="28.0" lower="-3.92" upper="0.78" velocity="3.2"/><!-- -225 deg to 45 deg -->
+    <dynamics damping="0.0" friction="0.0"/>
+  </joint>
+  <link name="wrist_1_link">
+    <visual>
+      <geometry>
+        <mesh filename="package://egomo_ur5/meshes/ur5/visual/wrist_1.dae"/>
       </geometry>
       <material name="LightGrey">
@@ -303,35 +206,5 @@
       </material>
     </visual>
-     <inertial>
-        <origin xyz="0 0 0" rpy="0 0 0" />
-        <mass value="1" />
-        <inertia
-          ixx="1.0" ixy="0.0" ixz="0.0"
-          iyy="1.0" iyz="0.0"
-          izz="1.0" />
-    </inertial>
-  </link>
-  <joint name="wrist_1_joint" type="revolute">
-    <parent link="forearm_link"/>
-    <child link="wrist_1_linka"/>
-    <!--origin xyz="0.0 0.0 ${forearm_length}" rpy="0.0 ${pi / 2.0} 0.0" /-->
- <origin  xyz="0.0 0.0 ${ur5_d4-wrist_1_length}" rpy="0.0 0.0 ${theta_4}"/>
-    <!--origin rpy="0.0 1.570796326795 0.0" xyz="0.0 0.0 0.39225"/-->
-    <axis xyz="0 0 -1"/>
-    <limit effort="28.0" lower="-3.92" upper="0.78" velocity="3.2"/><!-- -225 deg to 45 deg -->
-    <dynamics damping="0.0" friction="0.0"/>
-  </joint>
-  <link name="wrist_1_linka">
-    <visual>
-<origin xyz="0 0 0" rpy="-${pi/2} 0 0" />
-      <geometry>
-        <mesh filename="package://egomo_ur5/meshes/ur5/visual/wrist_1.dae"/>
-      </geometry>
-      <material name="LightGrey">
-        <color rgba="0.7 0.7 0.7 1.0"/>
-      </material>
-    </visual>
-    <collision>
-<origin xyz="0 0 0" rpy="-${pi/2} 0 0" />
+    <collision>
       <geometry>
         <mesh filename="package://egomo_ur5/meshes/ur5/collision/wrist_1.stl"/>
@@ -344,13 +217,17 @@
     </inertial>
   </link>
-<joint name="wrist_1_joint_F" type="fixed"> <!--Joint 1-->
-    <parent link="wrist_1_linka"/>
-    <child link="wrist_1_link"/>
-    <origin rpy="${alpha_4} 0.0 0.0" xyz="${ur5_a4} 0.0 0.0"/><!--origin rpy="0.0 0.0 0.7853981625" xyz="0.0 0.0 0.089159"/-->
-  </joint>
-  <link name="wrist_1_link">
-        <visual>
-      <geometry>
-        <box size="0 0 0" />
+  <joint name="wrist_2_joint" type="revolute">
+    <parent link="wrist_1_link"/>
+    <child link="wrist_2_link"/>
+    <!--origin rpy="0.0 0.0 0.0" xyz="0.0 0.093 0.0"/-->
+      <origin xyz="0.0 ${wrist_1_length} 0.0" rpy="0.0 0.0 0.0" />
+    <axis xyz="0 0 1"/>
+    <limit effort="28.0" lower="-${pi}" upper="${pi}" velocity="3.15"/>
+    <dynamics damping="0.0" friction="0.0"/>
+  </joint>
+  <link name="wrist_2_link">
+    <visual>
+      <geometry>
+        <mesh filename="package://egomo_ur5/meshes/ur5/visual/wrist_2.dae"/>
       </geometry>
       <material name="LightGrey">
@@ -358,58 +235,5 @@
       </material>
     </visual>
-     <inertial>
-        <origin xyz="0 0 0" rpy="0 0 0" />
-        <mass value="1" />
-        <inertia
-          ixx="1.0" ixy="0.0" ixz="0.0"
-          iyy="1.0" iyz="0.0"
-          izz="1.0" />
-    </inertial>
-  </link>
-<joint name="wrist_2_joint" type="revolute">
-    <parent link="wrist_1_link"/>
-    <child link="wrist_2_linka"/>
-    <!--origin rpy="0.0 0.0 0.0" xyz="0.0 0.093 0.0"/-->
-      <!--origin xyz="0.0 ${wrist_1_length} 0.0" rpy="0.0 0.0 0.0" /-->
- <origin rpy="0.0 0.0 ${theta_5}" xyz="0.0 ${-wrist_1_length}  ${ur5_d5-wrist_2_length}"/>
-    <axis xyz="0 0 -1"/>
-    <limit effort="28.0" lower="-${pi}" upper="${pi}" velocity="3.15"/>
-    <dynamics damping="0.0" friction="0.0"/>
-  </joint>
-  <link name="wrist_2_linka">
-        <visual>
-      <geometry>
-        <box size="0 0 0" />
-      </geometry>
-      <material name="LightGrey">
-        <color rgba="0.7 0.7 0.7 1.0"/>
-      </material>
-    </visual>
-     <inertial>
-        <origin xyz="0 0 0" rpy="0 0 0" />
-        <mass value="1" />
-        <inertia
-          ixx="1.0" ixy="0.0" ixz="0.0"
-          iyy="1.0" iyz="0.0"
-          izz="1.0" />
-    </inertial>
-  </link>
-<joint name="wrist_2_joint_F" type="fixed"> <!--Joint 1-->
-    <parent link="wrist_2_linka"/>
-    <child link="wrist_2_link"/>
-    <origin rpy="${alpha_5} 0.0 0.0" xyz="${ur5_a5} 0.0 0.0"/><!--origin rpy="0.0 0.0 0.7853981625" xyz="0.0 0.0 0.089159"/-->
-</joint>
-  <link name="wrist_2_link">
- <visual>
-<origin xyz="0 0 0" rpy="-${pi/2} 0 0" />
-      <geometry>
-        <mesh filename="package://egomo_ur5/meshes/ur5/visual/wrist_2.dae"/>
-      </geometry>
-      <material name="LightGrey">
-        <color rgba="0.7 0.7 0.7 1.0"/>
-      </material>
-    </visual>
-    <collision>
-<origin xyz="0 0 0" rpy="-${pi/2} 0 0" />
+    <collision>
       <geometry>
         <mesh filename="package://egomo_ur5/meshes/ur5/collision/wrist_2.stl"/>
@@ -421,19 +245,18 @@
       <inertia ixx="0.111172755531" ixy="0.0" ixz="0.0" iyy="0.111172755531" iyz="0.0" izz="0.21942"/>
     </inertial>
- </link>
-<joint name="wrist_3_joint" type="revolute">
+  </link>
+  <joint name="wrist_3_joint" type="revolute">
     <parent link="wrist_2_link"/>
-    <child link="wrist_3_linka"/>
+    <child link="wrist_3_link"/>
     <!--origin rpy="0.0 0.0 0.0" xyz="0.0 0.0 0.09465"/-->
-      <!--origin xyz="0.0 0.0 ${wrist_2_length}" rpy="0.0 0.0 0.0" /-->
- <origin rpy="0.0 0.0 ${theta_6}" xyz="0.0 ${wrist_2_length} ${ur5_d6-wrist_3_length}"/>
-    <axis xyz="0 0 -1"/>
+      <origin xyz="0.0 0.0 ${wrist_2_length}" rpy="0.0 0.0 0.0" />
+    <axis xyz="0 1 0"/>
     <limit effort="28.0" lower="-${pi}" upper="${pi}" velocity="3.15"/>
     <dynamics damping="0.0" friction="0.0"/>
   </joint>
-  <link name="wrist_3_linka">
-       <visual>
-      <geometry>
-        <box size="0 0 0" />
+  <link name="wrist_3_link">
+    <visual>
+      <geometry>
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