Commit message: Fixed problem with gripper model

File: egomo_ur5/urdf/ur5_egomo_table.urdf (robot description, URDF)
Before this commit: robot ur5, 24 links, 23 joints
Joints:
- joint robotiq_85_finger_left_1_joint: mimic joint=robotiq_85_finger_right_1_joint multiplier=-1 offset=0 -> joint=robotiq_85_finger_right_1_joint multiplier=1 offset=0; origin xyz=0.0305864 0 0.0549191 rpy=0 0 0 -> xyz=-0.0305864 0 0.0549191 rpy=0 0 0; type continuous -> revolute
- joint robotiq_85_finger_left_2_joint: origin xyz=0.0315367 0 -0.0037599 rpy=0 0 0 -> xyz=-0.0315367 0 -0.0037599 rpy=0 0 0
- joint robotiq_85_finger_left_3_joint: mimic joint=robotiq_85_finger_right_1_joint multiplier=-1 offset=0 -> joint=robotiq_85_finger_right_1_joint multiplier=1 offset=0; origin xyz=0.0127161 0 0.0613987 rpy=0 0 0 -> xyz=-0.0127161 0 0.0613987 rpy=0 0 0; type continuous -> revolute
- joint robotiq_85_finger_left_4_joint: mimic joint=robotiq_85_finger_right_1_joint multiplier=1 offset=0 -> joint=robotiq_85_finger_right_1_joint multiplier=-1 offset=0; origin xyz=0.0371331 0 0.0434428 rpy=0 0 0 -> xyz=-0.0371331 0 0.0434428 rpy=0 0 0; type continuous -> revolute
- joint robotiq_85_finger_right_1_joint: axis 0 1 0 -> 0 -1 0; origin xyz=-0.0305864 0 0.0549191 rpy=0 0 0 -> xyz=0.0305864 0 0.0549191 rpy=0 0 0; type continuous -> revolute
- joint robotiq_85_finger_right_2_joint: origin xyz=-0.0315367 0 -0.0037599 rpy=0 0 0 -> xyz=0.0315367 0 -0.0037599 rpy=0 0 0
- joint robotiq_85_finger_right_3_joint: mimic joint=robotiq_85_finger_right_1_joint multiplier=1 offset=0 -> joint=robotiq_85_finger_right_1_joint multiplier=-1 offset=0; origin xyz=-0.0127161 0 0.0613987 rpy=0 0 0 -> xyz=0.0127161 0 0.0613987 rpy=0 0 0; type continuous -> revolute
- joint robotiq_85_finger_right_4_joint: mimic joint=robotiq_85_finger_right_1_joint multiplier=-1 offset=0 -> joint=robotiq_85_finger_right_1_joint multiplier=1 offset=0; origin xyz=-0.0371331 0 0.0434428 rpy=0 0 0 -> xyz=0.0371331 0 0.0434428 rpy=0 0 0; type continuous -> revolute

Commit message: start to modularize

File: egomo_ur5/urdf/ur5_egomo_table.urdf (robot description, URDF)
Before this commit: robot ur5, 24 links, 23 joints
Links:
- added link forearm_linka, mass 2.275; collision mesh filename=package://egomo_ur5/meshes/ur5/collision/forearm.stl; visual mesh filename=package://egomo_ur5/meshes/ur5/visual/forearm.dae
- added link shoulder_linka, mass 3.7; collision mesh filename=package://egomo_ur5/meshes/ur5/collision/shoulder.stl; visual mesh filename=package://egomo_ur5/meshes/ur5/visual/shoulder.dae
- added link upper_arm_linka, mass 8.393; collision mesh filename=package://egomo_ur5/meshes/ur5/collision/upper_arm.stl; visual mesh filename=package://egomo_ur5/meshes/ur5/visual/upper_arm.dae
- added link wrist_1_linka, mass 1.219; collision mesh filename=package://egomo_ur5/meshes/ur5/collision/wrist_1.stl; visual mesh filename=package://egomo_ur5/meshes/ur5/visual/wrist_1.dae
- added link wrist_2_linka, mass 1; visual box size=0 0 0
- added link wrist_3_linka, mass 1; visual box size=0 0 0
- link forearm_link: mass 2.275 -> 1; geometry visual box size=0 0 0
- link shoulder_link: mass 3.7 -> 1; geometry visual box size=0 0 0
- link upper_arm_link: mass 8.393 -> 1; geometry visual box size=0 0 0
- link wrist_1_link: mass 1.219 -> 1; geometry visual box size=0 0 0
Joints:
- added joint elbow_joint_F: type fixed, parent forearm_linka, child forearm_link, origin xyz=0.39225 0.0   0.0 rpy=-0.00944871 0.0 0.0
- added joint shoulder_pan_joint_F: type fixed, parent shoulder_linka, child shoulder_link, origin xyz=0.0 0.0 0.0 rpy=1.57718 0.0 0.0
- added joint upper_arm_link_F: type fixed, parent upper_arm_linka, child upper_arm_link, origin xyz=0.425 0.0  0.0  rpy=-0.00201947 0.0 0.0
- added joint wrist_1_joint_F: type fixed, parent wrist_1_linka, child wrist_1_link, origin xyz=0.0 0.0 0.0 rpy=1.57342 0.0 0.0
- added joint wrist_2_joint_F: type fixed, parent wrist_2_linka, child wrist_2_link, origin xyz=0.0 0.0  0.0 rpy=-1.57255 0.0 0.0
- added joint wrist_3_joint_F: type fixed, parent wrist_3_linka, child wrist_3_link, origin xyz= 0.0 0.0  0.0 rpy=3.14331 0.0 0.0
- joint ee_fixed_joint: axis (none) -> 0 0 1; origin xyz=0.0 0.0823 0.0 rpy=-1.570796326795 0.0 0 -> xyz=0.0 0.0 0.0 rpy=0.0 0.0 0.0
- joint elbow_joint: axis 0 1 0 -> 0 0 -1; child forearm_link -> forearm_linka; origin xyz=0.0 -0.1197 0.425 rpy=0.0 0.0 0.0 -> xyz=0.0 0.0 0.0 rpy=0.0 0.0 -0.000189364
- joint shoulder_lift_joint: axis 0 1 0 -> 0 0 -1; child upper_arm_link -> upper_arm_linka; origin xyz=0.0 0.13585 0.0 rpy=0.0 1.570796326795 0.0 -> xyz=0.0 0.0 0.0 rpy=0.0 0.0 -0.000123686
- joint shoulder_pan_joint: child shoulder_link -> shoulder_linka; limit lower=-3.14159265 upper=3.14159265 effort=150.0 velocity=3.15 -> lower=-1.14159265 upper=1.14159265 effort=150.0 velocity=3.15; origin xyz=0.0 0.0 0.089159 rpy=0.0 0.0 0.0 -> xyz=0.0 0.0 0.089159 rpy=0.0 0.0 -0.00205442
- joint wrist_1_joint: axis 0 1 0 -> 0 0 -1; child wrist_1_link -> wrist_1_linka; origin xyz=0.0 0.0 0.39225 rpy=0.0 1.57079632679 0.0 -> xyz=0.0 0.0 -0.10915 rpy=0.0 0.0 0.000488426
- joint wrist_2_joint: child wrist_2_link -> wrist_2_linka; origin xyz=0.0 0.093 0.0 rpy=0.0 0.0 0.0 -> xyz=0.0 0.0  0.09465 rpy=0.0 0.0 -0.000123914
- joint wrist_3_joint: axis 0 1 0 -> 0 0 -1; child wrist_3_link -> wrist_3_linka; origin xyz=0.0 0.0 0.09465 rpy=0.0 0.0 0.0 -> xyz=0.0 0.0 -0.0823 rpy=0.0 0.0 3.14254
- joint wrist_3_link-tool0_fixed_joint: origin xyz=0 0.0823 0 rpy=-1.570796326795 0 0 -> xyz=0 0.0 0.0 rpy=0  0 0

File: egomo_ur5/urdf/ur5_egomo_table.urdf.xacro (robot description, xacro)
@@ -42,4 +42,5 @@
   <property name="wrist_2_cog" value="0.0 0.0018 0.11099" />
   <property name="wrist_3_cog" value="0.0 0.001159 0.0" />
+  <xacro:include filename="$(find egomo_ur5)/urdf/default_ur5_DH_parameters.xacro" />
   <!-- Kinematic model -->
   <!-- Properties from urcontrol.conf -->
@@ -88,28 +89,4 @@
 Joint 5(theta, d, a, alpha)3.14254 -0.0823 0 3.14331
 -->
-  <property name="theta_1" value="-0.00205442" />
-  <property name="ur5_d1" value="0.089159" />
-  <property name="ur5_a1" value="0.0" />
-  <property name="alpha_1" value="1.57718" />
-  <property name="theta_2" value="-0.000123686" />
-  <property name="ur5_d2" value="0.0" />
-  <property name="ur5_a2" value="0.42500" />
-  <property name="alpha_2" value="-0.00201947" />
-  <property name="theta_3" value="-0.000189364" />
-  <property name="ur5_d3" value="0.0" />
-  <property name="ur5_a3" value="0.39225" />
-  <property name="alpha_3" value="-0.00944871" />
-  <property name="theta_4" value="0.000488426" />
-  <property name="ur5_d4" value="-0.10915" />
-  <property name="ur5_a4" value="0.0" />
-  <property name="alpha_4" value="1.57342" />
-  <property name="theta_5" value="-0.000123914" />
-  <property name="ur5_d5" value="0.09465" />
-  <property name="ur5_a5" value="0.0" />
-  <property name="alpha_5" value="-1.57255" />
-  <property name="theta_6" value="3.14254" />
-  <property name="ur5_d6" value="-0.0823" />
-  <property name="ur5_a6" value="0.0" />
-  <property name="alpha_6" value="3.14331" />
  <!-- Arbitrary offsets for shoulder/elbow joints -->
   <property name="shoulder_offset" value="0.13585" />  <!-- measured from model -->
@@ -160,5 +137,5 @@
     <origin rpy="0.0 0.0 ${theta_1 }" xyz="0.0 0.0 ${ur5_d1}"/><!--origin rpy="0.0 0.0 0.7853981625" xyz="0.0 0.0 0.089159"/-->
     <axis xyz="0 0 1"/>
-    <limit effort="150.0" lower="-3.14159265" upper="3.14159265" velocity="3.15"/>
+    <limit effort="150.0" lower="-1.14159265" upper="1.14159265" velocity="3.15"/>
     <dynamics damping="0.0" friction="0.0"/>
   </joint>
