Commit message: relaxed limits in shoulder pan joint

File: egomo_ur5/urdf/ur5_robot.urdf.xacro (robot description, xacro)
@@ -102,5 +102,5 @@
         <!--origin rpy="0.0 0.0 0.7853981625" xyz="0.0 0.0 0.089159"/-->
         <axis xyz="0 0 1" />
-        <limit effort="150.0" lower="-1.14159265" upper="1.14159265" velocity="3.15" />
+        <limit effort="150.0" lower="-3.14159265" upper="3.14159265" velocity="3.15" />
         <dynamics damping="0.0" friction="0.0" />
     </joint>

Commit message: relaxed jointlimits in wristjoints

File: egomo_ur5/urdf/ur5_robot.urdf.xacro (robot description, xacro)
@@ -258,5 +258,6 @@
         <origin xyz="0.0 0.0 ${ur5_d4}" rpy="0.0 0.0 ${theta_4}" />
         <axis xyz="0 0 -1" />
-        <limit effort="28.0" lower="-3.92" upper="0.78" velocity="3.2" />
+        <!--limit effort="28.0" lower="-3.92" upper="0.78" velocity="3.2" /-->
+        <limit effort="28.0" lower="-${pi}" upper="${pi}" velocity="3.2" />
         <!-- -225 deg to 45 deg -->
         <dynamics damping="0.0" friction="0.0" />
@@ -361,5 +362,5 @@
         <origin rpy="0.0 0.0 ${theta_6}" xyz="0.0 0.0 ${ur5_d6}" />
         <axis xyz="0 0 -1" />
-        <limit effort="28.0" lower="-${pi}" upper="${pi}" velocity="3.15" />
+        <limit effort="28.0" lower="-${1.277*pi}" upper="${1.277*pi}" velocity="3.15" />
         <dynamics damping="0.0" friction="0.0" />
     </joint>
