Commit message: fixed new urdf file. TESTED WITH REAL ROBOT

File: egomo_ur5/urdf/ur5_egomo_table.urdf.xacro (robot description, xacro)
@@ -54,18 +54,19 @@
     center_of_mass = [ [0, -0.02561, 0.00193], [0.2125, 0, 0.11336], [0.11993, 0.0, 0.0265], [0, -0.0018, 0.01634], [0, 0.0018,0.01634], [0, 0, -0.001159] ]
   -->
+<!--
   <property name="theta_1" value="0.0" />
   <property name="ur5_d1" value="0.089159" />
   <property name="ur5_a1" value="0.0" />
   <property name="alpha_1" value="${pi/2}" />
-  <property name="theta_2" value="-${pi/2}" />
+  <property name="theta_2" value="0.0" />
   <property name="ur5_d2" value="0.0" />
-  <property name="ur5_a2" value="-0.42500" />
+  <property name="ur5_a2" value="0.425" />
   <property name="alpha_2" value="0.0" />
   <property name="theta_3" value="0.0" />
   <property name="ur5_d3" value="0.0" />
-  <property name="ur5_a3" value="-0.39225" />
+  <property name="ur5_a3" value="0.39225" />
   <property name="alpha_3" value="0.0" />
-  <property name="theta_4" value="-${pi/2}" />
-  <property name="ur5_d4" value="0.10915" />
+  <property name="theta_4" value="0.0" />
+  <property name="ur5_d4" value="-0.10915" />
   <property name="ur5_a4" value="0.0" />
   <property name="alpha_4" value="${pi/2}" />
@@ -74,8 +75,9 @@
   <property name="ur5_a5" value="0.0" />
   <property name="alpha_5" value="-${pi/2}" />
-  <property name="theta_6" value="0.0" />
-  <property name="ur5_d6" value="0.0823" />
+  <property name="theta_6" value="${pi}" />
+  <property name="ur5_d6" value="-0.0823" />
   <property name="ur5_a6" value="0.0" />
-  <property name="alpha_6" value="0.0" />
+  <property name="alpha_6" value="${pi}" />
+-->
 <!--
 Joint 0(theta, d, a, alpha)-0.00205442 0.089159 0 1.57718
@@ -85,4 +87,5 @@
 Joint 4(theta, d, a, alpha)-0.000123914 0.09465 0 -1.57255
 Joint 5(theta, d, a, alpha)3.14254 -0.0823 0 3.14331
+-->
   <property name="theta_1" value="-0.00205442" />
   <property name="ur5_d1" value="0.089159" />
@@ -97,5 +100,5 @@
   <property name="ur5_a3" value="0.39225" />
   <property name="alpha_3" value="-0.00944871" />
-  <property name="theta_4" value="-0.000488426" />
+  <property name="theta_4" value="0.000488426" />
   <property name="ur5_d4" value="-0.10915" />
   <property name="ur5_a4" value="0.0" />
@@ -109,13 +112,12 @@
   <property name="ur5_a6" value="0.0" />
   <property name="alpha_6" value="3.14331" />
--->
  <!-- Arbitrary offsets for shoulder/elbow joints -->
   <property name="shoulder_offset" value="0.13585" />  <!-- measured from model -->
-  <property name="elbow_offset" value="-0.1197" /> <!-- measured from model -->
+  <property name="elbow_offset" value="0.1197" /> <!-- measured from model -->
   <!-- link lengths used in model -->
   <property name="shoulder_height" value="${ur5_d1}" />
   <property name="upper_arm_length" value="${-ur5_a2}" />
   <property name="forearm_length" value="${-ur5_a3}" />
-  <property name="wrist_1_length" value="${ur5_d4 - elbow_offset - shoulder_offset}" />
+  <property name="wrist_1_length" value="${ur5_d4  + shoulder_offset+ elbow_offset}" />
   <property name="wrist_2_length" value="${ur5_d5}" />
   <property name="wrist_3_length" value="${ur5_d6}" />
@@ -163,5 +165,5 @@
   <link name="shoulder_linka">
     <visual>
-	<origin xyz="0 0 0" rpy="0.0 0 0" />
+	<origin xyz="0 0 0.0" rpy="0.0 0 0" />
       <geometry>
         <mesh filename="package://egomo_ur5/meshes/ur5/visual/shoulder.dae"/>
@@ -208,5 +210,5 @@
     <parent link="shoulder_link"/>
     <child link="upper_arm_linka"/>
- <origin rpy="0.0 0.0 ${theta_2}" xyz="0.0 0.0 ${ur5_d2+elbow_offset}"/><!--Joint 2-->
+ <origin rpy="0.0 0.0 ${theta_2}" xyz="0.0 0.0 ${ur5_d2}"/><!--Joint 2-->
     <axis xyz="0 0 -1"/>
     <limit effort="150.0" lower="-3.14159265" upper="-0.1" velocity="3.15"/>
@@ -215,5 +217,5 @@
   <link name="upper_arm_linka">
     <visual>
-	<origin xyz="0 0 0" rpy="-${pi/2} 0 0" />
+	<origin xyz="0 0 ${-shoulder_offset}" rpy="${pi/2} ${pi} ${pi/2}" />
       <geometry>
         <mesh filename="package://egomo_ur5/meshes/ur5/visual/upper_arm.dae"/>
@@ -224,5 +226,5 @@
     </visual>
     <collision>
-<origin xyz="0 0 0" rpy="-${pi/2} 0 0" />
+		<origin xyz="0 0 ${-shoulder_offset}" rpy="${pi/2} ${pi} ${pi/2}" />
       <geometry>
         <mesh filename="package://egomo_ur5/meshes/ur5/collision/upper_arm.stl"/>
@@ -238,5 +240,5 @@
     <parent link="upper_arm_linka"/>
     <child link="upper_arm_link"/>
-    <origin rpy="${alpha_2} 0.0 0.0" xyz="0.0 ${-ur5_a2} 0.0 "/><!--origin rpy="0.0 0.0 0.7853981625" xyz="0.0 0.0 0.089159"/-->
+    <origin rpy="${alpha_2} 0.0 0.0" xyz="${ur5_a2} 0.0  0.0 "/><!--origin rpy="0.0 0.0 0.7853981625" xyz="0.0 0.0 0.089159"/-->
   </joint>
   <link name="upper_arm_link">
@@ -261,5 +263,5 @@
     <parent link="upper_arm_link"/>
     <child link="forearm_linka"/>
- <origin rpy="0.0 0.0 ${theta_3}" xyz="0.0 0.0 ${ur5_d3-elbow_offset}"/>
+ <origin rpy="0.0 0.0 ${theta_3}" xyz="0.0 0.0 ${ur5_d3}"/>
 <!--origin rpy="0.0 0.0 0.0" xyz="0.0 -0.1197 0.425"/-->
     <axis xyz="0 0 -1"/>
@@ -269,5 +271,5 @@
 <link name="forearm_linka">
  <visual>
-	<origin xyz="0 0 0" rpy="-${pi/2} 0 0" />
+	<origin xyz="0 0 ${elbow_offset-shoulder_offset}" rpy="${pi/2} ${pi} ${pi/2}" />
       <geometry>
         <mesh filename="package://egomo_ur5/meshes/ur5/visual/forearm.dae"/>
@@ -278,5 +280,5 @@
     </visual>
     <collision>
-<origin xyz="0 0 0" rpy="-${pi/2} 0 0" />
+<origin xyz="0 0 ${elbow_offset-shoulder_offset}" rpy="${pi/2} ${pi} ${pi/2}" />
       <geometry>
         <mesh filename="package://egomo_ur5/meshes/ur5/collision/forearm.stl"/>
@@ -292,5 +294,5 @@
     <parent link="forearm_linka"/>
     <child link="forearm_link"/>
-    <origin rpy="${alpha_3} 0.0 0.0" xyz="0.0 ${-ur5_a3} 0.0"/><!--origin rpy="0.0 0.0 0.7853981625" xyz="0.0 0.0 0.089159"/-->
+    <origin rpy="${alpha_3} 0.0 0.0" xyz="${ur5_a3} 0.0   0.0"/><!--origin rpy="0.0 0.0 0.7853981625" xyz="0.0 0.0 0.089159"/-->
   </joint>
   <link name="forearm_link">
@@ -316,5 +318,5 @@
     <child link="wrist_1_linka"/>
     <!--origin xyz="0.0 0.0 ${forearm_length}" rpy="0.0 ${pi / 2.0} 0.0" /-->
- <origin  xyz="0.0 0.0 ${ur5_d4-wrist_1_length}" rpy="0.0 0.0 ${theta_4}"/>
+ <origin  xyz="0.0 0.0 ${ur5_d4}" rpy="0.0 0.0 ${theta_4}"/>
     <!--origin rpy="0.0 1.570796326795 0.0" xyz="0.0 0.0 0.39225"/-->
     <axis xyz="0 0 -1"/>
@@ -324,5 +326,5 @@
   <link name="wrist_1_linka">
     <visual>
-<origin xyz="0 0 0" rpy="-${pi/2} 0 0" />
+		<origin xyz="0 0 ${0.10915+(elbow_offset-shoulder_offset)}" rpy="${pi/2}  ${pi} 0" />
       <geometry>
         <mesh filename="package://egomo_ur5/meshes/ur5/visual/wrist_1.dae"/>
@@ -333,5 +335,5 @@
     </visual>
     <collision>
-<origin xyz="0 0 0" rpy="-${pi/2} 0 0" />
+		<origin xyz="0 0 ${0.10915+(elbow_offset-shoulder_offset)}" rpy="${pi/2}  ${pi} 0" />
       <geometry>
         <mesh filename="package://egomo_ur5/meshes/ur5/collision/wrist_1.stl"/>
@@ -372,6 +374,6 @@
     <!--origin rpy="0.0 0.0 0.0" xyz="0.0 0.093 0.0"/-->
       <!--origin xyz="0.0 ${wrist_1_length} 0.0" rpy="0.0 0.0 0.0" /-->
- <origin rpy="0.0 0.0 ${theta_5}" xyz="0.0 ${-wrist_1_length}  ${ur5_d5-wrist_2_length}"/>
-    <axis xyz="0 0 -1"/>
+ <origin rpy="0.0 0.0 ${theta_5}" xyz="0.0 0.0  ${ur5_d5}"/>
+    <axis xyz="0 0 1"/>
     <limit effort="28.0" lower="-${pi}" upper="${pi}" velocity="3.15"/>
     <dynamics damping="0.0" friction="0.0"/>
@@ -398,9 +400,9 @@
     <parent link="wrist_2_linka"/>
     <child link="wrist_2_link"/>
-    <origin rpy="${alpha_5} 0.0 0.0" xyz="${ur5_a5} 0.0 0.0"/><!--origin rpy="0.0 0.0 0.7853981625" xyz="0.0 0.0 0.089159"/-->
+    <origin rpy="${alpha_5} 0.0 0.0" xyz="${ur5_a5} 0.0  0.0"/><!--origin rpy="0.0 0.0 0.7853981625" xyz="0.0 0.0 0.089159"/-->
 </joint>
   <link name="wrist_2_link">
  <visual>
-<origin xyz="0 0 0" rpy="-${pi/2} 0 0" />
+<origin xyz="0 0.09465 0" rpy="-${pi/2} 0 ${pi}" />
       <geometry>
         <mesh filename="package://egomo_ur5/meshes/ur5/visual/wrist_2.dae"/>
@@ -411,5 +413,5 @@
     </visual>
     <collision>
-<origin xyz="0 0 0" rpy="-${pi/2} 0 0" />
+<origin xyz="0 0.09465 0" rpy="-${pi/2} 0 ${pi}" />
       <geometry>
         <mesh filename="package://egomo_ur5/meshes/ur5/collision/wrist_2.stl"/>
@@ -427,5 +429,5 @@
     <!--origin rpy="0.0 0.0 0.0" xyz="0.0 0.0 0.09465"/-->
       <!--origin xyz="0.0 0.0 ${wrist_2_length}" rpy="0.0 0.0 0.0" /-->
- <origin rpy="0.0 0.0 ${theta_6}" xyz="0.0 ${wrist_2_length} ${ur5_d6-wrist_3_length}"/>
+ <origin rpy="0.0 0.0 ${theta_6}" xyz="0.0 0.0 ${ur5_d6}"/>
     <axis xyz="0 0 -1"/>
     <limit effort="28.0" lower="-${pi}" upper="${pi}" velocity="3.15"/>
@@ -453,9 +455,9 @@
     <parent link="wrist_3_linka"/>
     <child link="wrist_3_link"/>
-    <origin rpy="${alpha_6} 0.0 0.0" xyz="${ur5_a6} 0.0 0.0"/><!--origin rpy="0.0 0.0 0.7853981625" xyz="0.0 0.0 0.089159"/-->
+    <origin rpy="${alpha_6} 0.0 0.0" xyz=" ${ur5_a6} 0.0  0.0"/><!--origin rpy="0.0 0.0 0.7853981625" xyz="0.0 0.0 0.089159"/-->
   </joint>
   <link name="wrist_3_link">
      <visual>
-	<origin xyz="0 0 0" rpy="-${pi/2} 0 0" />
+	<origin xyz="0 0 -0.0823" rpy="-${pi/2} ${pi} ${pi}" />
       <geometry>
         <mesh filename="package://egomo_ur5/meshes/ur5/visual/wrist_3.dae"/>
@@ -466,5 +468,5 @@
     </visual>
     <collision>
-<origin xyz="0 0 0" rpy="-${pi/2} 0 0" />
+<origin xyz="0 0 -0.0823" rpy="-${pi/2} ${pi} ${pi}" />
       <geometry>
         <mesh filename="package://egomo_ur5/meshes/ur5/collision/wrist_3.stl"/>
@@ -548,17 +550,18 @@
     </actuator>
   </transmission>
+    <!--
   <link name="base"/>
   <joint name="base_link-base_fixed_joint" type="fixed">
-    <!-- NOTE: this rotation is only needed as long as base_link itself is
+     NOTE: this rotation is only needed as long as base_link itself is
                  not corrected wrt the real robot (ie: rotated over 180
                  degrees)
-      -->
     <origin rpy="0 0 -3.14159265" xyz="0 0 0"/>
     <parent link="base_link"/>
     <child link="base"/>
   </joint>
+ -->
   <link name="tool0"/>
   <joint name="wrist_3_link-tool0_fixed_joint" type="fixed">
-    <origin rpy="${pi}  0 0" xyz="0 0.0 -0.0823"/>
+    <origin rpy="0  0 0" xyz="0 0.0 0.0"/>
     <parent link="wrist_3_link"/>
     <child link="tool0"/>
@@ -579,5 +582,5 @@
     </inertial>
     <visual>
-      <origin rpy="0 ${pi} -1.570796326795" xyz="0 0 0.0375"/>
+      <origin rpy="0 3.14159265359 -1.570796326795" xyz="0 0 0.0375"/>
       <geometry>
         <mesh filename="package://egomo_ur5/meshes/robotiq-ft300/visual/ft300.dae"/>
@@ -585,5 +588,5 @@
     </visual>
     <collision>
-      <origin rpy="0 ${pi} -1.570796326795" xyz="0 0 0.0375"/>
+      <origin rpy="0 3.14159265359 -1.570796326795" xyz="0 0 0.0375"/>
       <geometry>
         <mesh filename="package://egomo_ur5/meshes/robotiq-ft300/collision/ft300.stl"/>
