Commit message: structured urdf files with new xacros.

File: egomo_ur5/urdf/ur5_egomo_table.urdf.xacro (robot description, xacro)
@@ -1,839 +1,26 @@
-<?xml version="1.0" ?>
-<!-- =================================================================================== -->
-<!-- |    This document was autogenerated by xacro from ur5_joint_limited_robot.urdf.xacro | -->
-<!-- |    EDITING THIS FILE BY HAND IS NOT RECOMMENDED                                 | -->
-<!-- =================================================================================== -->
-<robot name="ur5" xmlns:xacro="http://www.ros.org/wiki/xacro">
-  <!-- ur5 arm -->
- <!-- common stuff -->
-  <gazebo>
-    <plugin filename="libgazebo_ros_control.so" name="ros_control">
-      <!--robotNamespace>/UR5/</robotNamespace-->
-      <!--robotSimType>gazebo_ros_control/DefaultRobotHWSim</robotSimType-->
-    </plugin>
-    <!--
-    <plugin name="gazebo_ros_power_monitor_controller" filename="libgazebo_ros_power_monitor.so">
-      <alwaysOn>true</alwaysOn>
-      <updateRate>1.0</updateRate>
-      <timeout>5</timeout>
-      <powerStateTopic>power_state</powerStateTopic>
-      <powerStateRate>10.0</powerStateRate>
-      <fullChargeCapacity>87.78</fullChargeCapacity>
-      <dischargeRate>-474</dischargeRate>
-      <chargeRate>525</chargeRate>
-      <dischargeVoltage>15.52</dischargeVoltage>
-      <chargeVoltage>16.41</chargeVoltage>
-    </plugin>
--->
-  </gazebo>
-<property name="pi" value="3.1415926535898" />3.14159265359
-  <!-- Inertia parameters -->
-  <property name="base_mass" value="4.0" />  <!-- This mass might be incorrect -->
-  <property name="shoulder_mass" value="3.7000" />
-  <property name="upper_arm_mass" value="8.3930" />
-  <property name="forearm_mass" value="2.2750" />
-  <property name="wrist_1_mass" value="1.2190" />
-  <property name="wrist_2_mass" value="1.2190" />
-  <property name="wrist_3_mass" value="0.1879" />
-  <property name="shoulder_cog" value="0.0 0.00193 -0.02561" />
-  <property name="upper_arm_cog" value="0.0 -0.024201 0.2125" />
-  <property name="forearm_cog" value="0.0 0.0265 0.11993" />
-  <property name="wrist_1_cog" value="0.0 0.110949 0.01634" />
-  <property name="wrist_2_cog" value="0.0 0.0018 0.11099" />
-  <property name="wrist_3_cog" value="0.0 0.001159 0.0" />
-  <xacro:include filename="$(find egomo_ur5)/urdf/default_ur5_DH_parameters.xacro" />
-  <!-- Kinematic model -->
-  <!-- Properties from urcontrol.conf -->
-  <!--
-    DH for UR5:
-    a = [0.00000, -0.42500, -0.39225,  0.00000,  0.00000,  0.0000]
-    d = [0.089159,  0.00000,  0.00000,  0.10915,  0.09465,  0.0823]
-    alpha = [ 1.570796327, 0, 0, 1.570796327, -1.570796327, 0 ]
-    theta = [0, -1.570796327, 0, -1.570796327, 0, 0]
-    joint_direction = [-1, -1, 1, 1, 1, 1]
-    mass = [3.7000, 8.3930, 2.2750, 1.2190, 1.2190, 0.1879]
-    center_of_mass = [ [0, -0.02561, 0.00193], [0.2125, 0, 0.11336], [0.11993, 0.0, 0.0265], [0, -0.0018, 0.01634], [0, 0.0018,0.01634], [0, 0, -0.001159] ]
-  -->
-<!--
-  <property name="theta_1" value="0.0" />
-  <property name="ur5_d1" value="0.089159" />
-  <property name="ur5_a1" value="0.0" />
-  <property name="alpha_1" value="${pi/2}" />
-  <property name="theta_2" value="0.0" />
-  <property name="ur5_d2" value="0.0" />
-  <property name="ur5_a2" value="0.425" />
-  <property name="alpha_2" value="0.0" />
-  <property name="theta_3" value="0.0" />
-  <property name="ur5_d3" value="0.0" />
-  <property name="ur5_a3" value="0.39225" />
-  <property name="alpha_3" value="0.0" />
-  <property name="theta_4" value="0.0" />
-  <property name="ur5_d4" value="-0.10915" />
-  <property name="ur5_a4" value="0.0" />
-  <property name="alpha_4" value="${pi/2}" />
-  <property name="theta_5" value="0.0" />
-  <property name="ur5_d5" value="0.09465" />
-  <property name="ur5_a5" value="0.0" />
-  <property name="alpha_5" value="-${pi/2}" />
-  <property name="theta_6" value="${pi}" />
-  <property name="ur5_d6" value="-0.0823" />
-  <property name="ur5_a6" value="0.0" />
-  <property name="alpha_6" value="${pi}" />
--->
-<!--
-Joint 0(theta, d, a, alpha)-0.00205442 0.089159 0 1.57718
-Joint 1(theta, d, a, alpha)-0.000123686 0 0.425 -0.00201947
-Joint 2(theta, d, a, alpha)-0.000189364 0 0.39225 -0.00944871
-Joint 3(theta, d, a, alpha)0.000488426 -0.10915 0 1.57342
-Joint 4(theta, d, a, alpha)-0.000123914 0.09465 0 -1.57255
-Joint 5(theta, d, a, alpha)3.14254 -0.0823 0 3.14331
--->
- <!-- Arbitrary offsets for shoulder/elbow joints -->
-  <property name="shoulder_offset" value="0.13585" />  <!-- measured from model -->
-  <property name="elbow_offset" value="0.1197" /> <!-- measured from model -->
-  <!-- link lengths used in model -->
-  <property name="shoulder_height" value="${ur5_d1}" />
-  <property name="upper_arm_length" value="${-ur5_a2}" />
-  <property name="forearm_length" value="${-ur5_a3}" />
-  <property name="wrist_1_length" value="${ur5_d4  + shoulder_offset+ elbow_offset}" />
-  <property name="wrist_2_length" value="${ur5_d5}" />
-  <property name="wrist_3_length" value="${ur5_d6}" />
-  <!--property name="shoulder_height" value="0.089159" /-->
-  <!--property name="shoulder_offset" value="0.13585" /-->  <!-- shoulder_offset - elbow_offset + wrist_1_length = 0.10915 -->
-  <!--property name="upper_arm_length" value="0.42500" /-->
-  <!--property name="elbow_offset" value="0.1197" /-->       <!-- CAD measured -->
-  <!--property name="forearm_length" value="0.39225" /-->
-  <!--property name="wrist_1_length" value="0.093" /-->     <!-- CAD measured -->
-  <!--property name="wrist_2_length" value="0.09465" /-->   <!-- In CAD this distance is 0.930, but in the spec it is 0.09465 -->
-  <!--property name="wrist_3_length" value="0.0823" /-->
-  <property name="shoulder_radius" value="0.060" />   <!-- manually measured -->
-  <property name="upper_arm_radius" value="0.054" />  <!-- manually measured -->
-  <property name="elbow_radius" value="0.060" />      <!-- manually measured -->
-  <property name="forearm_radius" value="0.040" />    <!-- manually measured -->
-  <property name="wrist_radius" value="0.045" />      <!-- manually measured -->
-  <link name="base_link">
-    <visual>
-      <geometry>
-        <mesh filename="package://egomo_ur5/meshes/ur5/visual/base.dae"/>
-      </geometry>
-      <material name="LightGrey">
-        <color rgba="0.7 0.7 0.7 1.0"/>
-      </material>
-    </visual>
-    <collision>
-      <geometry>
-        <mesh filename="package://egomo_ur5/meshes/ur5/collision/base.stl"/>
-      </geometry>
-    </collision>
-    <inertial>
-      <mass value="4.0"/>
-      <origin rpy="0 0 0" xyz="0.0 0.0 0.0"/>
-      <inertia ixx="0.00443333156" ixy="0.0" ixz="0.0" iyy="0.00443333156" iyz="0.0" izz="0.0072"/>
-    </inertial>
-  </link>
-  <joint name="shoulder_pan_joint" type="revolute"> <!--Joint 1-->
-    <parent link="base_link"/>
-    <child link="shoulder_linka"/>
-    <origin rpy="0.0 0.0 ${theta_1 }" xyz="0.0 0.0 ${ur5_d1}"/><!--origin rpy="0.0 0.0 0.7853981625" xyz="0.0 0.0 0.089159"/-->
-    <axis xyz="0 0 1"/>
-    <limit effort="150.0" lower="-1.14159265" upper="1.14159265" velocity="3.15"/>
-    <dynamics damping="0.0" friction="0.0"/>
-  </joint>
-  <link name="shoulder_linka">
-    <visual>
-	<origin xyz="0 0 0.0" rpy="0.0 0 0" />
-      <geometry>
-        <mesh filename="package://egomo_ur5/meshes/ur5/visual/shoulder.dae"/>
-      </geometry>
-      <material name="LightGrey">
-        <color rgba="0.7 0.7 0.7 1.0"/>
-      </material>
-    </visual>
-    <collision>
-      <geometry>
-        <mesh filename="package://egomo_ur5/meshes/ur5/collision/shoulder.stl"/>
-      </geometry>
-    </collision>
-    <inertial>
-      <mass value="3.7"/>
-      <origin rpy="0 0 0" xyz="0.0 0.0 0.0"/>
-      <inertia ixx="0.010267495893" ixy="0.0" ixz="0.0" iyy="0.010267495893" iyz="0.0" izz="0.00666"/>
-    </inertial>
-  </link>
- <joint name="shoulder_pan_joint_F" type="fixed"> <!--Joint 1-->
-    <parent link="shoulder_linka"/>
-    <child link="shoulder_link"/>
-    <origin rpy="${alpha_1} 0.0 0.0" xyz="${ur5_a1} 0.0 0.0"/><!--origin rpy="0.0 0.0 0.7853981625" xyz="0.0 0.0 0.089159"/-->
-  </joint>
-  <link name="shoulder_link">
-    <visual>
-      <geometry>
-        <box size="0 0 0" />
-      </geometry>
-      <material name="LightGrey">
-        <color rgba="0.7 0.7 0.7 1.0"/>
-      </material>
-    </visual>
-     <inertial>
+<?xml version="1.0"?>
+<robot name="egomo_ur5" xmlns:xacro="http://www.ros.org/wiki/xacro">
+    <xacro:include filename="$(find egomo_ur5)/urdf/ur5_robot.urdf.xacro" />
+    <xacro:include filename="$(find egomo_ur5)/urdf/egomo_sensor.urdf.xacro" />
+    <xacro:include filename="$(find egomo_ur5)/urdf/robotiq_85_gripper.urdf.xacro" />
+    <link name="world" />
+    <!-- ==============add UR5 robot arm=================== -->
+    <xacro:ur5 prefix="" parent="world">
         <origin xyz="0 0 0" rpy="0 0 0" />
-        <mass value="1" />
-        <inertia
-          ixx="1.0" ixy="0.0" ixz="0.0"
-          iyy="1.0" iyz="0.0"
-          izz="1.0" />
-    </inertial>
-  </link>
-  <joint name="shoulder_lift_joint" type="revolute"><!--Joint 2-->
-    <parent link="shoulder_link"/>
-    <child link="upper_arm_linka"/>
- <origin rpy="0.0 0.0 ${theta_2}" xyz="0.0 0.0 ${ur5_d2}"/><!--Joint 2-->
-    <axis xyz="0 0 -1"/>
-    <limit effort="150.0" lower="-3.14159265" upper="-0.1" velocity="3.15"/>
-    <dynamics damping="0.0" friction="0.0"/>
-  </joint>
-  <link name="upper_arm_linka">
-    <visual>
-	<origin xyz="0 0 ${-shoulder_offset}" rpy="${pi/2} ${pi} ${pi/2}" />
-      <geometry>
-        <mesh filename="package://egomo_ur5/meshes/ur5/visual/upper_arm.dae"/>
-      </geometry>
-      <material name="LightGrey">
-        <color rgba="0.7 0.7 0.7 1.0"/>
-      </material>
-    </visual>
-    <collision>
-		<origin xyz="0 0 ${-shoulder_offset}" rpy="${pi/2} ${pi} ${pi/2}" />
-      <geometry>
-        <mesh filename="package://egomo_ur5/meshes/ur5/collision/upper_arm.stl"/>
-      </geometry>
-    </collision>
-    <inertial>
-      <mass value="8.393"/>
-      <origin rpy="0 0 0" xyz="0.0 0.0 0.28"/>
-      <inertia ixx="0.22689067591" ixy="0.0" ixz="0.0" iyy="0.22689067591" iyz="0.0" izz="0.0151074"/>
-    </inertial>
-  </link>
-<joint name="upper_arm_link_F" type="fixed"> <!--Joint 1-->
-    <parent link="upper_arm_linka"/>
-    <child link="upper_arm_link"/>
-    <origin rpy="${alpha_2} 0.0 0.0" xyz="${ur5_a2} 0.0  0.0 "/><!--origin rpy="0.0 0.0 0.7853981625" xyz="0.0 0.0 0.089159"/-->
-  </joint>
-  <link name="upper_arm_link">
-    <visual>
-      <geometry>
-        <box size="0 0 0" />
-      </geometry>
-      <material name="LightGrey">
-        <color rgba="0.7 0.7 0.7 1.0"/>
-      </material>
-    </visual>
-     <inertial>
-        <origin xyz="0 0 0" rpy="0 0 0" />
-        <mass value="1" />
-        <inertia
-          ixx="1.0" ixy="0.0" ixz="0.0"
-          iyy="1.0" iyz="0.0"
-          izz="1.0" />
-    </inertial>
-  </link>
-  <joint name="elbow_joint" type="revolute"> <!--Joint 3-->
-    <parent link="upper_arm_link"/>
-    <child link="forearm_linka"/>
- <origin rpy="0.0 0.0 ${theta_3}" xyz="0.0 0.0 ${ur5_d3}"/>
-<!--origin rpy="0.0 0.0 0.0" xyz="0.0 -0.1197 0.425"/-->
-    <axis xyz="0 0 -1"/>
-    <limit effort="150.0" lower="-3" upper="3" velocity="3.15"/> <!-- +/- 175 deg -->
-    <dynamics damping="0.0" friction="0.0"/>
-  </joint>
-<link name="forearm_linka">
- <visual>
-	<origin xyz="0 0 ${elbow_offset-shoulder_offset}" rpy="${pi/2} ${pi} ${pi/2}" />
-      <geometry>
-        <mesh filename="package://egomo_ur5/meshes/ur5/visual/forearm.dae"/>
-      </geometry>
-      <material name="LightGrey">
-        <color rgba="0.7 0.7 0.7 1.0"/>
-      </material>
-    </visual>
-    <collision>
-<origin xyz="0 0 ${elbow_offset-shoulder_offset}" rpy="${pi/2} ${pi} ${pi/2}" />
-      <geometry>
-        <mesh filename="package://egomo_ur5/meshes/ur5/collision/forearm.stl"/>
-      </geometry>
-    </collision>
-    <inertial>
-      <mass value="2.275"/>
-      <origin rpy="0 0 0" xyz="0.0 0.0 0.25"/>
-      <inertia ixx="0.049443313556" ixy="0.0" ixz="0.0" iyy="0.049443313556" iyz="0.0" izz="0.004095"/>
-    </inertial>
- </link>
-<joint name="elbow_joint_F" type="fixed"> <!--Joint 1-->
-    <parent link="forearm_linka"/>
-    <child link="forearm_link"/>
-    <origin rpy="${alpha_3} 0.0 0.0" xyz="${ur5_a3} 0.0   0.0"/><!--origin rpy="0.0 0.0 0.7853981625" xyz="0.0 0.0 0.089159"/-->
-  </joint>
-  <link name="forearm_link">
-    <visual>
-      <geometry>
-        <box size="0 0 0" />
-      </geometry>
-      <material name="LightGrey">
-        <color rgba="0.7 0.7 0.7 1.0"/>
-      </material>
-    </visual>
-     <inertial>
-        <origin xyz="0 0 0" rpy="0 0 0" />
-        <mass value="1" />
-        <inertia
-          ixx="1.0" ixy="0.0" ixz="0.0"
-          iyy="1.0" iyz="0.0"
-          izz="1.0" />
-    </inertial>
-  </link>
-  <joint name="wrist_1_joint" type="revolute">
-    <parent link="forearm_link"/>
-    <child link="wrist_1_linka"/>
-    <!--origin xyz="0.0 0.0 ${forearm_length}" rpy="0.0 ${pi / 2.0} 0.0" /-->
- <origin  xyz="0.0 0.0 ${ur5_d4}" rpy="0.0 0.0 ${theta_4}"/>
-    <!--origin rpy="0.0 1.570796326795 0.0" xyz="0.0 0.0 0.39225"/-->
-    <axis xyz="0 0 -1"/>
-    <limit effort="28.0" lower="-3.92" upper="0.78" velocity="3.2"/><!-- -225 deg to 45 deg -->
-    <dynamics damping="0.0" friction="0.0"/>
-  </joint>
-  <link name="wrist_1_linka">
-    <visual>
-		<origin xyz="0 0 ${0.10915+(elbow_offset-shoulder_offset)}" rpy="${pi/2}  ${pi} 0" />
-      <geometry>
-        <mesh filename="package://egomo_ur5/meshes/ur5/visual/wrist_1.dae"/>
-      </geometry>
-      <material name="LightGrey">
-        <color rgba="0.7 0.7 0.7 1.0"/>
-      </material>
-    </visual>
-    <collision>
-		<origin xyz="0 0 ${0.10915+(elbow_offset-shoulder_offset)}" rpy="${pi/2}  ${pi} 0" />
-      <geometry>
-        <mesh filename="package://egomo_ur5/meshes/ur5/collision/wrist_1.stl"/>
-      </geometry>
-    </collision>
-    <inertial>
-      <mass value="1.219"/>
-      <origin rpy="0 0 0" xyz="0.0 0.0 0.0"/>
-      <inertia ixx="0.111172755531" ixy="0.0" ixz="0.0" iyy="0.111172755531" iyz="0.0" izz="0.21942"/>
-    </inertial>
-  </link>
-<joint name="wrist_1_joint_F" type="fixed"> <!--Joint 1-->
-    <parent link="wrist_1_linka"/>
-    <child link="wrist_1_link"/>
-    <origin rpy="${alpha_4} 0.0 0.0" xyz="${ur5_a4} 0.0 0.0"/><!--origin rpy="0.0 0.0 0.7853981625" xyz="0.0 0.0 0.089159"/-->
-  </joint>
-  <link name="wrist_1_link">
-        <visual>
-      <geometry>
-        <box size="0 0 0" />
-      </geometry>
-      <material name="LightGrey">
-        <color rgba="0.7 0.7 0.7 1.0"/>
-      </material>
-    </visual>
-     <inertial>
-        <origin xyz="0 0 0" rpy="0 0 0" />
-        <mass value="1" />
-        <inertia
-          ixx="1.0" ixy="0.0" ixz="0.0"
-          iyy="1.0" iyz="0.0"
-          izz="1.0" />
-    </inertial>
-  </link>
-<joint name="wrist_2_joint" type="revolute">
-    <parent link="wrist_1_link"/>
-    <child link="wrist_2_linka"/>
-    <!--origin rpy="0.0 0.0 0.0" xyz="0.0 0.093 0.0"/-->
-      <!--origin xyz="0.0 ${wrist_1_length} 0.0" rpy="0.0 0.0 0.0" /-->
- <origin rpy="0.0 0.0 ${theta_5}" xyz="0.0 0.0  ${ur5_d5}"/>
-    <axis xyz="0 0 1"/>
-    <limit effort="28.0" lower="-${pi}" upper="${pi}" velocity="3.15"/>
-    <dynamics damping="0.0" friction="0.0"/>
-  </joint>
-  <link name="wrist_2_linka">
-        <visual>
-      <geometry>
-        <box size="0 0 0" />
-      </geometry>
-      <material name="LightGrey">
-        <color rgba="0.7 0.7 0.7 1.0"/>
-      </material>
-    </visual>
-     <inertial>
-        <origin xyz="0 0 0" rpy="0 0 0" />
-        <mass value="1" />
-        <inertia
-          ixx="1.0" ixy="0.0" ixz="0.0"
-          iyy="1.0" iyz="0.0"
-          izz="1.0" />
-    </inertial>
-  </link>
-<joint name="wrist_2_joint_F" type="fixed"> <!--Joint 1-->
-    <parent link="wrist_2_linka"/>
-    <child link="wrist_2_link"/>
-    <origin rpy="${alpha_5} 0.0 0.0" xyz="${ur5_a5} 0.0  0.0"/><!--origin rpy="0.0 0.0 0.7853981625" xyz="0.0 0.0 0.089159"/-->
-</joint>
-  <link name="wrist_2_link">
- <visual>
-<origin xyz="0 0.09465 0" rpy="-${pi/2} 0 ${pi}" />
-      <geometry>
-        <mesh filename="package://egomo_ur5/meshes/ur5/visual/wrist_2.dae"/>
-      </geometry>
-      <material name="LightGrey">
-        <color rgba="0.7 0.7 0.7 1.0"/>
-      </material>
-    </visual>
-    <collision>
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
Commit message: moved tool0 to gripper tip

File: egomo_ur5/urdf/ur5_egomo_table.urdf.xacro (robot description, xacro)
@@ -12,10 +12,10 @@
     <link name="tool0" />
     <joint name="wrist_3_link-tool0_fixed_joint" type="fixed">
-        <origin rpy="0  0 0" xyz="0 0.0 0.0" />
+        <origin rpy="0  0 0" xyz="0 0.0 0.2" />
         <parent link="wrist_3_link" />
         <child link="tool0" />
     </joint>
     <!-- ==============add EGOMO senor component=============== -->
-    <xacro:egomo_sensor prefix="" parent="tool0">
+    <xacro:egomo_sensor prefix="" parent="wrist_3_link">
         <origin xyz="0 0 0.011" rpy="0 0 0" />
     </xacro:egomo_sensor>
