Commit message: corrected xacro definition

File: egomo_ur5/urdf/default_egomo_sensor_parameters.xacro (robot description, xacro)
@@ -1,4 +1,4 @@
 <?xml version="1.0"?>
-<robot xmlns:xacro="http://www.ros.org/wiki/xacro">
+<robot xmlns:xacro="http://ros.org/wiki/xacro">
 <xacro:property name="egomo_side_cam_origin">
   <origin rpy="-2.4191 -1.5692 0.1464" xyz="0.0151 0.0696 0.0558" />

File: egomo_ur5/urdf/default_ur5_DH_parameters.xacro (robot description, xacro)
@@ -1,4 +1,4 @@
 <?xml version="1.0"?>
-<robot xmlns:xacro="http://www.ros.org/wiki/xacro">
+<robot xmlns:xacro="http://ros.org/wiki/xacro">
     <property name="theta_1" value="-0.00205442" />
     <property name="ur5_d1" value="0.089159" />

File: egomo_ur5/urdf/ur5_egomo_table.urdf.xacro (robot description, xacro)
@@ -1,4 +1,4 @@
 <?xml version="1.0"?>
-<robot name="egomo_ur5" xmlns:xacro="http://www.ros.org/wiki/xacro">
+<robot name="egomo_ur5" xmlns:xacro="http://ros.org/wiki/xacro">
     <xacro:include filename="$(find egomo_ur5)/urdf/ur5_robot.urdf.xacro" />
     <xacro:include filename="$(find egomo_ur5)/urdf/egomo_sensor.urdf.xacro" />
@@ -9,11 +9,4 @@
         <origin xyz="0 0 0" rpy="0 0 0" />
     </xacro:ur5>
-    <!-- ==============add tool0 for moveit naming convention=========== -->
-    <link name="tool0" />
-    <joint name="wrist_3_link-tool0_fixed_joint" type="fixed">
-        <origin rpy="0  0 0" xyz="0 0.0 0.2" />
-        <parent link="wrist_3_link" />
-        <child link="tool0" />
-    </joint>
     <!-- ==============add EGOMO senor component=============== -->
     <xacro:egomo_sensor prefix="" parent="wrist_3_link">
@@ -24,3 +17,10 @@
         <origin xyz="0 0 -0.003" rpy="0 0 0" />
     </xacro:robotiq_85_gripper>
+    <!-- ==============add tool0 for moveit naming convention=========== -->
+    <link name="tool0" />
+    <joint name="fts_toolside-tool0_fixed_joint" type="fixed">
+        <origin rpy="0  0 0" xyz="0 0.0 0.175" />
+        <parent link="fts_toolside" />
+        <child link="tool0" />
+    </joint>
 </robot>

File: egomo_ur5/urdf/ur5_robot.urdf.xacro (robot description, xacro)
@@ -4,5 +4,5 @@
 <!-- |    EDITING THIS FILE BY HAND IS NOT RECOMMENDED                                 | -->
 <!-- =================================================================================== -->
-<robot name="ur5" xmlns:xacro="http://www.ros.org/wiki/xacro">
+<robot name="ur5" xmlns:xacro="http://ros.org/wiki/xacro">
 <xacro:include filename="$(find egomo_ur5)/urdf/default_ur5_DH_parameters.xacro" />
     <xacro:property name="pi" value="3.1415926535898" />
