Commit message: eliminated most of the xacro warnings

File: egomo_ur5/urdf/default_ur5_DH_parameters.xacro (robot description, xacro)
@@ -1,27 +1,27 @@
 <?xml version="1.0"?>
 <robot xmlns:xacro="http://ros.org/wiki/xacro">
-    <property name="theta_1" value="-0.00205442" />
-    <property name="ur5_d1" value="0.089159" />
-    <property name="ur5_a1" value="0.0" />
-    <property name="alpha_1" value="1.57718" />
-    <property name="theta_2" value="-0.000123686" />
-    <property name="ur5_d2" value="0.0" />
-    <property name="ur5_a2" value="0.42500" />
-    <property name="alpha_2" value="-0.00201947" />
-    <property name="theta_3" value="-0.000189364" />
-    <property name="ur5_d3" value="0.0" />
-    <property name="ur5_a3" value="0.39225" />
-    <property name="alpha_3" value="-0.00944871" />
-    <property name="theta_4" value="0.000488426" />
-    <property name="ur5_d4" value="-0.10915" />
-    <property name="ur5_a4" value="0.0" />
-    <property name="alpha_4" value="1.57342" />
-    <property name="theta_5" value="-0.000123914" />
-    <property name="ur5_d5" value="0.09465" />
-    <property name="ur5_a5" value="0.0" />
-    <property name="alpha_5" value="-1.57255" />
-    <property name="theta_6" value="3.14254" />
-    <property name="ur5_d6" value="-0.0823" />
-    <property name="ur5_a6" value="0.0" />
-    <property name="alpha_6" value="3.14331" />
+    <xacro:property name="theta_1" value="-0.00205442" />
+    <xacro:property name="ur5_d1" value="0.089159" />
+    <xacro:property name="ur5_a1" value="0.0" />
+    <xacro:property name="alpha_1" value="1.57718" />
+    <xacro:property name="theta_2" value="-0.000123686" />
+    <xacro:property name="ur5_d2" value="0.0" />
+    <xacro:property name="ur5_a2" value="0.42500" />
+    <xacro:property name="alpha_2" value="-0.00201947" />
+    <xacro:property name="theta_3" value="-0.000189364" />
+    <xacro:property name="ur5_d3" value="0.0" />
+    <xacro:property name="ur5_a3" value="0.39225" />
+    <xacro:property name="alpha_3" value="-0.00944871" />
+    <xacro:property name="theta_4" value="0.000488426" />
+    <xacro:property name="ur5_d4" value="-0.10915" />
+    <xacro:property name="ur5_a4" value="0.0" />
+    <xacro:property name="alpha_4" value="1.57342" />
+    <xacro:property name="theta_5" value="-0.000123914" />
+    <xacro:property name="ur5_d5" value="0.09465" />
+    <xacro:property name="ur5_a5" value="0.0" />
+    <xacro:property name="alpha_5" value="-1.57255" />
+    <xacro:property name="theta_6" value="3.14254" />
+    <xacro:property name="ur5_d6" value="-0.0823" />
+    <xacro:property name="ur5_a6" value="0.0" />
+    <xacro:property name="alpha_6" value="3.14331" />
 </robot>

File: egomo_ur5/urdf/egomo_sensor.urdf.xacro (robot description, xacro)
@@ -3,5 +3,5 @@
     <xacro:include filename="$(find egomo_ur5)/urdf/default_egomo_sensor_parameters.xacro" />
     <xacro:macro name="egomo_sensor" params="prefix parent *origin">
-        <property name="pi" value="3.1415926535898" />
+        <xacro:property name="pi" value="3.1415926535898" />
         <!-- ========================================== -->
         <!-- Mount the force torque sensor (fts) to the robot -->
